File: NJM2903_Non-inverting_comparator_circuit_with_hysteresis.kicad_sch (KiCad schematic)
At the start: 9 parts, among them J101 from Sensor, J102 to M304, U101 NJM2903

Commit message: DOCs
Parts:
- added FL101: DSS1NB31H104Q91, symbol Device:Filter_EMI_LCL
- added unit 2 of U101
Connections:
- net GND: now also FL101.2
- net Vin: now also FL101.1; no longer U101.3 (+)
- new net: FL101.3, U101.3 (+)
- no-connect marks 0 -> 3
Other:
- moved on the sheet: J101

Commit message: continue モデル番号を変更する予定
Parts:
- added C1, C2, C3, C4: 0.1uF, Capacitor_THT:C_Disc_D3.4mm_W2.1mm_P2.50mm, symbol Device:C_Small
- FL1: renamed from FL101; footprint (none) -> holly:DSS1
- J1: renamed from J101; footprint (none) -> Connector_JST:JST_XH_B2B-XH-A_1x02_P2.50mm_Vertical
- J2: renamed from J102; footprint (none) -> Connector_JST:JST_XH_B3B-XH-A_1x03_P2.50mm_Vertical
- R1: renamed from R101; footprint (none) -> Resistor_THT:R_Axial_DIN0207_L6.3mm_D2.5mm_P10.16mm_Horizontal
- R2: renamed from R102; footprint (none) -> Resistor_THT:R_Axial_DIN0207_L6.3mm_D2.5mm_P10.16mm_Horizontal
- R3: renamed from R103; footprint (none) -> Resistor_THT:R_Axial_DIN0207_L6.3mm_D2.5mm_P10.16mm_Horizontal
- R4: renamed from R104; footprint (none) -> Resistor_THT:R_Axial_DIN0207_L6.3mm_D2.5mm_P10.16mm_Horizontal
- U1: renamed from U101; footprint (none) -> Package_DIP:DIP-8_W7.62mm_LongPads
- V101, V102: now left out of the parts list
Connections:
- net +5V: now also C1.1, C2.1
- net GND: now also C1.2, C2.2, C3.2, C4.2
- net Vout: now also C3.1
- net at FL1.3, U1.3 (+): now also C4.1
Other:
- company: (none) -> YS-Lab
- title: (none) -> Voltage Amplifier & Comparator for CTT-10-CLS-CV-25
- moved on the sheet: FL1, R2, R3, U1B, U1C
